File: DCHY-P2-6464-1515-VP/led-panel-DCHY-P2-644-1515-VP.sch (KiCad schematic (older format))
At the start: 69 parts, among them T1 TC7258E, T2 TC7258E, T3 TC7258E, T4 TC7258E, T5 TC7258E, T6 TC7258E, T7 TC7258E, T8 TC7258E, U1 74HC245, U2 74HC245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

Commit message: Corrected row off by one mistakes.
Connections:
- net ROW_B32 is gone; now on net ROW_B31: T8.14 (O7)
- net ROW_B10: now also T6.5 (O2); no longer T6.4 (O1)
- net ROW_B11: now also T6.6 (O3); no longer T6.5 (O2)
- net ROW_B12: now also T6.11 (O4); no longer T6.6 (O3)
- net ROW_B13: now also T6.12 (O5); no longer T6.11 (O4)
- net ROW_B14: now also T6.13 (O6); no longer T6.12 (O5)
- net ROW_B15: now also T6.14 (O7); no longer T6.13 (O6)
- net ROW_B16: now also T7.3 (O0); no longer T6.14 (O7)
- net ROW_B17: now also T7.4 (O1); no longer T7.3 (O0)
- net ROW_B18: now also T7.5 (O2); no longer T7.4 (O1)
- net ROW_B19: now also T7.6 (O3); no longer T7.5 (O2)
- net ROW_B20: now also T7.11 (O4); no longer T7.6 (O3)
- net ROW_B21: now also T7.12 (O5); no longer T7.11 (O4)
- net ROW_B22: now also T7.13 (O6); no longer T7.12 (O5)
- net ROW_B23: now also T7.14 (O7); no longer T7.13 (O6)
- net ROW_B24: now also T8.3 (O0); no longer T7.14 (O7)
- net ROW_B25: now also T8.4 (O1); no longer T8.3 (O0)
- net ROW_B26: now also T8.5 (O2); no longer T8.4 (O1)
- net ROW_B27: now also T8.6 (O3); no longer T8.5 (O2)
- net ROW_B28: now also T8.11 (O4); no longer T8.6 (O3)
- net ROW_B29: now also T8.12 (O5); no longer T8.11 (O4)
- net ROW_B30: now also T8.13 (O6); no longer T8.12 (O5)
- net ROW_B31: no longer T8.13 (O6)
- net ROW_B9: now also T6.4 (O1); no longer T6.3 (O0)
- net ~ROW16-24EN: no longer T7.10 (ENL)
- net ~ROW25-32EN: no longer T8.10 (ENL)
- new net ~ROW16-23EN: T7.10 (ENL)
- new net ~ROW24-31EN: T8.10 (ENL)
Changed lines of the file:
@@
 ~ROW8-15EN
 Text Label 3700 13000 2    50   ~ 10
-~ROW16-24EN
+~ROW16-23EN
 Text Label 3700 14800 2    50   ~ 10
-~ROW25-32EN
+~ROW24-31EN
 Wire Wire Line
 	4800 1100 4900 1100
@@
 Wire Wire Line
 	4800 11200 4900 11200
-Text Label 4900 10500 0    50   ~ 10
+Text Label 4900 10600 0    50   ~ 10
 ROW_B9
-Text Label 4900 10600 0    50   ~ 10
+Text Label 4900 10700 0    50   ~ 10
 ROW_B10
-Text Label 4900 10700 0    50   ~ 10
+Text Label 4900 10800 0    50   ~ 10
 ROW_B11
-Text Label 4900 10800 0    50   ~ 10
+Text Label 4900 10900 0    50   ~ 10
 ROW_B12
-Text Label 4900 10900 0    50   ~ 10
+Text Label 4900 11000 0    50   ~ 10
 ROW_B13
-Text Label 4900 11000 0    50   ~ 10
+Text Label 4900 11100 0    50   ~ 10
 ROW_B14
-Text Label 4900 11100 0    50   ~ 10
+Text Label 4900 11200 0    50   ~ 10
 ROW_B15
-Text Label 4900 11200 0    50   ~ 10
+Text Label 4900 12300 0    50   ~ 10
 ROW_B16
 Wire Wire Line
@@
 Wire Wire Line
 	4800 13000 4900 13000
-Text Label 4900 12300 0    50   ~ 10
+Text Label 4900 12400 0    50   ~ 10
 ROW_B17
-Text Label 4900 12400 0    50   ~ 10
+Text Label 4900 12500 0    50   ~ 10
 ROW_B18
-Text Label 4900 12500 0    50   ~ 10
+Text Label 4900 12600 0    50   ~ 10
 ROW_B19
-Text Label 4900 12600 0    50   ~ 10
+Text Label 4900 12700 0    50   ~ 10
 ROW_B20
-Text Label 4900 12700 0    50   ~ 10
+Text Label 4900 12800 0    50   ~ 10
 ROW_B21
-Text Label 4900 12800 0    50   ~ 10
+Text Label 4900 12900 0    50   ~ 10
 ROW_B22
-Text Label 4900 12900 0    50   ~ 10
+Text Label 4900 13000 0    50   ~ 10
 ROW_B23
-Text Label 4900 13000 0    50   ~ 10
+Text Label 4900 14100 0    50   ~ 10
 ROW_B24
 Wire Wire Line
@@
 Wire Wire Line
 	4800 14800 4900 14800
-Text Label 4900 14100 0    50   ~ 10
+Text Label 4900 14200 0    50   ~ 10
 ROW_B25
-Text Label 4900 14200 0    50   ~ 10
+Text Label 4900 14300 0    50   ~ 10
 ROW_B26
-Text Label 4900 14300 0    50   ~ 10
+Text Label 4900 14400 0    50   ~ 10
 ROW_B27
-Text Label 4900 14400 0    50   ~ 10
+Text Label 4900 14500 0    50   ~ 10
 ROW_B28
-Text Label 4900 14500 0    50   ~ 10
+Text Label 4900 14600 0    50   ~ 10
 ROW_B29
-Text Label 4900 14600 0    50   ~ 10
+Text Label 4900 14700 0    50   ~ 10
 ROW_B30
-Text Label 4900 14700 0    50   ~ 10
+Text Label 4900 14800 0    50   ~ 10
 ROW_B31
-Text Label 4900 14800 0    50   ~ 10
-ROW_B32
 Wire Wire Line
 	6900 2050 6900 1950

Commit message: More off by one fixes.
Connections:
- net ROW_A32 is gone; now on net ROW_A31: T4.14 (O7)
- net ROW_A10: now also T2.5 (O2); no longer T2.4 (O1)
- net ROW_A11: now also T2.6 (O3); no longer T2.5 (O2)
- net ROW_A12: now also T2.11 (O4); no longer T2.6 (O3)
- net ROW_A13: now also T2.12 (O5); no longer T2.11 (O4)
- net ROW_A14: now also T2.13 (O6); no longer T2.12 (O5)
- net ROW_A15: now also T2.14 (O7); no longer T2.13 (O6)
- net ROW_A16: now also T3.3 (O0); no longer T2.14 (O7)
- net ROW_A17: now also T3.4 (O1); no longer T3.3 (O0)
- net ROW_A18: now also T3.5 (O2); no longer T3.4 (O1)
- net ROW_A19: now also T3.6 (O3); no longer T3.5 (O2)
- net ROW_A20: now also T3.11 (O4); no longer T3.6 (O3)
- net ROW_A21: now also T3.12 (O5); no longer T3.11 (O4)
- net ROW_A22: now also T3.13 (O6); no longer T3.12 (O5)
- net ROW_A23: now also T3.14 (O7); no longer T3.13 (O6)
- net ROW_A24: now also T4.3 (O0); no longer T3.14 (O7)
- net ROW_A25: now also T4.4 (O1); no longer T4.3 (O0)
- net ROW_A26: now also T4.5 (O2); no longer T4.4 (O1)
- net ROW_A27: now also T4.6 (O3); no longer T4.5 (O2)
- net ROW_A28: now also T4.11 (O4); no longer T4.6 (O3)
- net ROW_A29: now also T4.12 (O5); no longer T4.11 (O4)
- net ROW_A30: now also T4.13 (O6); no longer T4.12 (O5)
- net ROW_A31: no longer T4.13 (O6)
- net ROW_A9: now also T2.4 (O1); no longer T2.3 (O0)
- net ~ROW16-23EN: now also T3.10 (ENL)
- net ~ROW16-24EN: no longer T3.10 (ENL)
- net ~ROW24-31EN: now also T4.10 (ENL)
- net ~ROW25-32EN: no longer T4.10 (ENL)
- net ROW_B8: now reaches T6.3 (O0)
- new net ROW_A8: T2.3 (O0)
Changed lines of the file:
@@
 EESchema Schematic File Version 4
 LIBS:led-panel-DCHY-P2-644-1515-VP-cache
-EELAYER 29 0
+EELAYER 26 0
 EELAYER END
 $Descr A2 23386 16535
@@
 ~ROW8-15EN
 Text Label 3700 5400 2    50   ~ 10
-~ROW16-24EN
+~ROW16-23EN
 Text Label 3700 7200 2    50   ~ 10
-~ROW25-32EN
+~ROW24-31EN
 $Comp
 L led-panel-chipset:TC7258E T5
@@
 Wire Wire Line
 	4800 3600 4900 3600
-Text Label 4900 2900 0    50   ~ 10
-ROW_A9
 Text Label 4900 3000 0    50   ~ 10
-ROW_A10
+ROW_A9
 Text Label 4900 3100 0    50   ~ 10
-ROW_A11
+ROW_A10
 Text Label 4900 3200 0    50   ~ 10
-ROW_A12
+ROW_A11
 Text Label 4900 3300 0    50   ~ 10
-ROW_A13
+ROW_A12
 Text Label 4900 3400 0    50   ~ 10
-ROW_A14
+ROW_A13
 Text Label 4900 3500 0    50   ~ 10
-ROW_A15
+ROW_A14
 Text Label 4900 3600 0    50   ~ 10
+ROW_A15
+Text Label 4900 4700 0    50   ~ 10
 ROW_A16
 Wire Wire Line
@@
 Wire Wire Line
 	4800 5400 4900 5400
-Text Label 4900 4700 0    50   ~ 10
-ROW_A17
 Text Label 4900 4800 0    50   ~ 10
-ROW_A18
+ROW_A17
 Text Label 4900 4900 0    50   ~ 10
-ROW_A19
+ROW_A18
 Text Label 4900 5000 0    50   ~ 10
-ROW_A20
+ROW_A19
 Text Label 4900 5100 0    50   ~ 10
-ROW_A21
+ROW_A20
 Text Label 4900 5200 0    50   ~ 10
-ROW_A22
+ROW_A21
 Text Label 4900 5300 0    50   ~ 10
-ROW_A23
+ROW_A22
 Text Label 4900 5400 0    50   ~ 10
+ROW_A23
+Text Label 4900 6500 0    50   ~ 10
 ROW_A24
 Wire Wire Line
@@
 Wire Wire Line
 	4800 7200 4900 7200
-Text Label 4900 6500 0    50   ~ 10
-ROW_A25
 Text Label 4900 6600 0    50   ~ 10
-ROW_A26
+ROW_A25
 Text Label 4900 6700 0    50   ~ 10
-ROW_A27
+ROW_A26
 Text Label 4900 6800 0    50   ~ 10
-ROW_A28
+ROW_A27
 Text Label 4900 6900 0    50   ~ 10
-ROW_A29
+ROW_A28
 Text Label 4900 7000 0    50   ~ 10
-ROW_A30
+ROW_A29
 Text Label 4900 7100 0    50   ~ 10
-ROW_A31
+ROW_A30
 Text Label 4900 7200 0    50   ~ 10
-ROW_A32
+ROW_A31
 Wire Wire Line
 	4800 8700 4900 8700
@@
 Text Label 6900 13700 1    50   ~ 10
 COL_BB0
+Text Label 4900 2900 0    50   ~ 10
+ROW_A8
+Text Label 4900 10500 0    50   ~ 10
+ROW_B8
 $EndSCHEMATC
