File: P2-1515_1010-32S-JJ-V2.0/led-panel-P2-1515_1010-32S-JJ-V2.0.sch (KiCad schematic (older format))
At the start: 68 parts, among them T1 TC7258E, T2 TC7258E, T3 TC7258E, T4 TC7258E, T5 TC7258E, T6 TC7258E, T7 TC7258E, T8 TC7258E, U1 SM74HC04, U2 74HC245, U3 74HC245, U4 74HC245

Commit message: Corrected shift register part number.
Parts:
- BU1, BU2, BU3, BU4, BU5, BU6, BU7, BU8, GU1, GU2, GU3, GU4, GU5, GU6, GU7, GU8, RU1, RU2, RU3, RU4, RU5, RU6, RU7, RU8: value FM6126 -> ICN2037
Changed lines of the file:
@@
 P 7600 2550
 F 0 "GU1" V 7600 2600 50  0000 R CNN
-F 1 "FM6126" V 7500 2700 50  0000 R CNN
+F 1 "ICN2037" V 7500 2700 50  0000 R CNN
 F 2 "" H 7550 4600 50  0001 C CNN
 F 3 "" H 7550 4600 50  0001 C CNN
@@
 P 10000 2550
 F 0 "GU3" V 10000 2600 50  0000 R CNN
-F 1 "FM6126" V 9900 2700 50  0000 R CNN
+F 1 "ICN2037" V 9900 2700 50  0000 R CNN
 F 2 "" H 9950 4600 50  0001 C CNN
 F 3 "" H 9950 4600 50  0001 C CNN
@@
 P 12400 2550
 F 0 "GU5" V 12400 2600 50  0000 R CNN
-F 1 "FM6126" V 12300 2700 50  0000 R CNN
+F 1 "ICN2037" V 12300 2700 50  0000 R CNN
 F 2 "" H 12350 4600 50  0001 C CNN
 F 3 "" H 12350 4600 50  0001 C CNN
@@
 P 14800 2550
 F 0 "GU7" V 14800 2600 50  0000 R CNN
-F 1 "FM6126" V 14700 2700 50  0000 R CNN
+F 1 "ICN2037" V 14700 2700 50  0000 R CNN
 F 2 "" H 14750 4600 50  0001 C CNN
 F 3 "" H 14750 4600 50  0001 C CNN
@@
 P 7600 4550
 F 0 "RU1" V 7600 4600 50  0000 R CNN
-F 1 "FM6126" V 7500 4700 50  0000 R CNN
+F 1 "ICN2037" V 7500 4700 50  0000 R CNN
 F 2 "" H 7550 6600 50  0001 C CNN
 F 3 "" H 7550 6600 50  0001 C CNN
@@
 P 10000 4550
 F 0 "RU3" V 10000 4600 50  0000 R CNN
-F 1 "FM6126" V 9900 4700 50  0000 R CNN
+F 1 "ICN2037" V 9900 4700 50  0000 R CNN
 F 2 "" H 9950 6600 50  0001 C CNN
 F 3 "" H 9950 6600 50  0001 C CNN
@@
 P 12400 4550
 F 0 "RU5" V 12400 4600 50  0000 R CNN
-F 1 "FM6126" V 12300 4700 50  0000 R CNN
+F 1 "ICN2037" V 12300 4700 50  0000 R CNN
 F 2 "" H 12350 6600 50  0001 C CNN
 F 3 "" H 12350 6600 50  0001 C CNN
@@
 P 14800 4550
 F 0 "RU7" V 14800 4600 50  0000 R CNN
-F 1 "FM6126" V 14700 4700 50  0000 R CNN
+F 1 "ICN2037" V 14700 4700 50  0000 R CNN
 F 2 "" H 14750 6600 50  0001 C CNN
 F 3 "" H 14750 6600 50  0001 C CNN
@@
 P 12400 6550
 F 0 "BU5" V 12400 6600 50  0000 R CNN
-F 1 "FM6126" V 12300 6700 50  0000 R CNN
+F 1 "ICN2037" V 12300 6700 50  0000 R CNN
 F 2 "" H 12350 8600 50  0001 C CNN
 F 3 "" H 12350 8600 50  0001 C CNN
@@
 P 14800 6550
 F 0 "BU7" V 14800 6600 50  0000 R CNN
-F 1 "FM6126" V 14700 6700 50  0000 R CNN
+F 1 "ICN2037" V 14700 6700 50  0000 R CNN
 F 2 "" H 14750 8600 50  0001 C CNN
 F 3 "" H 14750 8600 50  0001 C CNN
@@
 P 7600 10300
 F 0 "GU2" V 7600 10350 50  0000 R CNN
-F 1 "FM6126" V 7500 10450 50  0000 R CNN
+F 1 "ICN2037" V 7500 10450 50  0000 R CNN
 F 2 "" H 7550 12350 50  0001 C CNN
 F 3 "" H 7550 12350 50  0001 C CNN
@@
 P 10000 10300
 F 0 "GU4" V 10000 10350 50  0000 R CNN
-F 1 "FM6126" V 9900 10450 50  0000 R CNN
+F 1 "ICN2037" V 9900 10450 50  0000 R CNN
 F 2 "" H 9950 12350 50  0001 C CNN
 F 3 "" H 9950 12350 50  0001 C CNN
@@
 P 12400 10300
 F 0 "GU6" V 12400 10350 50  0000 R CNN
-F 1 "FM6126" V 12300 10450 50  0000 R CNN
+F 1 "ICN2037" V 12300 10450 50  0000 R CNN
 F 2 "" H 12350 12350 50  0001 C CNN
 F 3 "" H 12350 12350 50  0001 C CNN
@@
 P 14800 10300
 F 0 "GU8" V 14800 10350 50  0000 R CNN
-F 1 "FM6126" V 14700 10450 50  0000 R CNN
+F 1 "ICN2037" V 14700 10450 50  0000 R CNN
 F 2 "" H 14750 12350 50  0001 C CNN
 F 3 "" H 14750 12350 50  0001 C CNN
@@
 P 7600 12300
 F 0 "RU2" V 7600 12350 50  0000 R CNN
-F 1 "FM6126" V 7500 12450 50  0000 R CNN
+F 1 "ICN2037" V 7500 12450 50  0000 R CNN
 F 2 "" H 7550 14350 50  0001 C CNN
 F 3 "" H 7550 14350 50  0001 C CNN
@@
 P 10000 12300
 F 0 "RU4" V 10000 12350 50  0000 R CNN
-F 1 "FM6126" V 9900 12450 50  0000 R CNN
+F 1 "ICN2037" V 9900 12450 50  0000 R CNN
 F 2 "" H 9950 14350 50  0001 C CNN
 F 3 "" H 9950 14350 50  0001 C CNN
@@
 P 12400 12300
 F 0 "RU6" V 12400 12350 50  0000 R CNN
-F 1 "FM6126" V 12300 12450 50  0000 R CNN
+F 1 "ICN2037" V 12300 12450 50  0000 R CNN
 F 2 "" H 12350 14350 50  0001 C CNN
 F 3 "" H 12350 14350 50  0001 C CNN
@@
 P 14800 12300
 F 0 "RU8" V 14800 12350 50  0000 R CNN
-F 1 "FM6126" V 14700 12450 50  0000 R CNN
+F 1 "ICN2037" V 14700 12450 50  0000 R CNN
 F 2 "" H 14750 14350 50  0001 C CNN
 F 3 "" H 14750 14350 50  0001 C CNN
@@
 P 7600 14300
 F 0 "BU2" V 7600 14350 50  0000 R CNN
-F 1 "FM6126" V 7500 14450 50  0000 R CNN
+F 1 "ICN2037" V 7500 14450 50  0000 R CNN
 F 2 "" H 7550 16350 50  0001 C CNN
 F 3 "" H 7550 16350 50  0001 C CNN
@@
 P 10000 14300
 F 0 "BU4" V 10000 14350 50  0000 R CNN
-F 1 "FM6126" V 9900 14450 50  0000 R CNN
+F 1 "ICN2037" V 9900 14450 50  0000 R CNN
 F 2 "" H 9950 16350 50  0001 C CNN
 F 3 "" H 9950 16350 50  0001 C CNN
@@
 P 12400 14300
 F 0 "BU6" V 12400 14350 50  0000 R CNN
-F 1 "FM6126" V 12300 14450 50  0000 R CNN
+F 1 "ICN2037" V 12300 14450 50  0000 R CNN
 F 2 "" H 12350 16350 50  0001 C CNN
 F 3 "" H 12350 16350 50  0001 C CNN
@@
 P 7600 6550
 F 0 "BU1" V 7600 6600 50  0000 R CNN
-F 1 "FM6126" V 7500 6700 50  0000 R CNN
+F 1 "ICN2037" V 7500 6700 50  0000 R CNN
 F 2 "" H 7550 8600 50  0001 C CNN
 F 3 "" H 7550 8600 50  0001 C CNN
@@
 P 10000 6550
 F 0 "BU3" V 10000 6600 50  0000 R CNN
-F 1 "FM6126" V 9900 6700 50  0000 R CNN
+F 1 "ICN2037" V 9900 6700 50  0000 R CNN
 F 2 "" H 9950 8600 50  0001 C CNN
 F 3 "" H 9950 8600 50  0001 C CNN
@@
 P 14800 14300
 F 0 "BU8" V 14800 14350 50  0000 R CNN
-F 1 "FM6126" V 14700 14450 50  0000 R CNN
+F 1 "ICN2037" V 14700 14450 50  0000 R CNN
 F 2 "" H 14750 16350 50  0001 C CNN
 F 3 "" H 14750 16350 50  0001 C CNN

Commit message: Some chip naming and signal corrections.
Thanks @smunaut :D
Parts:
- T1, T2, T3, T4, T5, T6, T7, T8: value TC7258E -> ICN2012
- U2, U3, U4: value 74HC245 -> ICN74HC245
- U2: value 74HC04 -> ICN74HC245
Connections:
- net A3out is gone; now on net A3: J?.12 (Pin_12)
Changed lines of the file:
@@
 P 1600 3600
 F 0 "U2" H 1350 4250 50  0000 C CNN
-F 1 "74HC245" H 1850 4250 50  0000 C CNN
+F 1 "ICN74HC245" H 1850 4250 50  0000 C CNN
 F 2 "" H 1600 3600 50  0001 C CNN
 F 3 "http://www.ti.com/lit/gpn/sn74HC245" H 1600 3600 50  0001 C CNN
@@
 P 1600 5700
 F 0 "U3" H 1350 6350 50  0000 C CNN
-F 1 "74HC245" H 1850 6350 50  0000 C CNN
+F 1 "ICN74HC245" H 1850 6350 50  0000 C CNN
 F 2 "" H 1600 5700 50  0001 C CNN
 F 3 "http://www.ti.com/lit/gpn/sn74HC245" H 1600 5700 50  0001 C CNN
@@
 P 1600 7800
 F 0 "U4" H 1350 8450 50  0000 C CNN
-F 1 "74HC245" H 1850 8450 50  0000 C CNN
+F 1 "ICN74HC245" H 1850 8450 50  0000 C CNN
 F 2 "" H 1600 7800 50  0001 C CNN
 F 3 "http://www.ti.com/lit/gpn/sn74HC245" H 1600 7800 50  0001 C CNN
@@
 A2
 Text Label 18600 8900 0    50   ~ 10
-A3out
+A3
 Text Label 18600 8700 0    50   ~ 10
 A4out
@@
 P 4300 6800
 F 0 "T4" H 4050 7250 50  0000 C CNN
-F 1 "TC7258E" H 4500 7250 50  0000 C CNN
+F 1 "ICN2012" H 4500 7250 50  0000 C CNN
 F 2 "" H 4300 7800 50  0001 C CNN
 F 3 "" H 4300 7800 50  0001 C CNN
@@
 P 4300 9000
 F 0 "T5" H 4050 9450 50  0000 C CNN
-F 1 "TC7258E" H 4500 9450 50  0000 C CNN
+F 1 "ICN2012" H 4500 9450 50  0000 C CNN
 F 2 "" H 4300 10000 50  0001 C CNN
 F 3 "" H 4300 10000 50  0001 C CNN
@@
 P 4300 10800
 F 0 "T6" H 4050 11250 50  0000 C CNN
-F 1 "TC7258E" H 4500 11250 50  0000 C CNN
+F 1 "ICN2012" H 4500 11250 50  0000 C CNN
 F 2 "" H 4300 11800 50  0001 C CNN
 F 3 "" H 4300 11800 50  0001 C CNN
@@
 P 4300 12600
 F 0 "T7" H 4050 13050 50  0000 C CNN
-F 1 "TC7258E" H 4500 13050 50  0000 C CNN
+F 1 "ICN2012" H 4500 13050 50  0000 C CNN
 F 2 "" H 4300 13600 50  0001 C CNN
 F 3 "" H 4300 13600 50  0001 C CNN
@@
 P 4300 14400
 F 0 "T8" H 4050 14850 50  0000 C CNN
-F 1 "TC7258E" H 4500 14850 50  0000 C CNN
+F 1 "ICN2012" H 4500 14850 50  0000 C CNN
 F 2 "" H 4300 15400 50  0001 C CNN
 F 3 "" H 4300 15400 50  0001 C CNN
@@
 P 1700 12200
 F 0 "U2" H 1700 12520 50  0000 C CNN
-F 1 "74HC04" H 1700 12427 50  0000 C CNN
+F 1 "ICN74HC245" H 1700 12427 50  0000 C CNN
 F 2 "" H 1700 12200 50  0001 C CNN
 F 3 "https://assets.nexperia.com/documents/data-sheet/74HC_HCT04.pdf" H 1700 12200 50  0001 C CNN
@@
 P 4300 3200
 F 0 "T2" H 4050 3650 50  0000 C CNN
-F 1 "TC7258E" H 4500 3650 50  0000 C CNN
+F 1 "ICN2012" H 4500 3650 50  0000 C CNN
 F 2 "" H 4300 4200 50  0001 C CNN
 F 3 "" H 4300 4200 50  0001 C CNN
@@
 P 4300 1400
 F 0 "T1" H 4050 1850 50  0000 C CNN
-F 1 "TC7258E" H 4500 1850 50  0000 C CNN
+F 1 "ICN2012" H 4500 1850 50  0000 C CNN
 F 2 "" H 4300 2400 50  0001 C CNN
 F 3 "" H 4300 2400 50  0001 C CNN
@@
 P 4300 5000
 F 0 "T3" H 4050 5450 50  0000 C CNN
-F 1 "TC7258E" H 4500 5450 50  0000 C CNN
+F 1 "ICN2012" H 4500 5450 50  0000 C CNN
 F 2 "" H 4300 6000 50  0001 C CNN
 F 3 "" H 4300 6000 50  0001 C CNN

Commit message: Added decoupling capacitors. Corrected current set resistors.
Parts:
- added C? (x36): 100n, symbol Device:C_Small
- added E? (x5): 220u, symbol Device:CP
- GR1, GR2, GR3, GR4, GR5, GR6, GR7, GR8: value 4k -> 4k12
- RR1, RR2, RR3, RR4, RR5, RR6, RR7, RR8: value ??? -> 7k5
Connections:
- net +5V: now also C?.1, C?.1, C?.1, C?.1, C?.1, C?.1, C?.1, C?.1, C?.1, C?.1, C?.1, C?.1, C?.1, C?.1, C?.1, C?.1, C?.1, C?.1, C?.1, C?.1, C?.1, C?.1, C?.1, C?.1, C?.2, C?.2, C?.2, C?.2, C?.2, C?.2, C?.2, C?.2, C?.2, C?.2, C?.2, C?.2, E?.1, E?.1, E?.1, E?.1, E?.1
- net GND: now also C?.1, C?.1, C?.1, C?.1, C?.1, C?.1, C?.1, C?.1, C?.1, C?.1, C?.1, C?.1, C?.2, C?.2, C?.2, C?.2, C?.2, C?.2, C?.2, C?.2, C?.2, C?.2, C?.2, C?.2, C?.2, C?.2, C?.2, C?.2, C?.2, C?.2, C?.2, C?.2, C?.2, C?.2, C?.2, C?.2, E?.2, E?.2, E?.2, E?.2, E?.2
Other:
- moved on the sheet: U1A, U1B, U1C, U1D, U1E, U1G, U2, U2F, U3, U4
